File: DS2482 1 Wire Controller/Ds2482/DS2482 1 Wire Controller Rev C.brd (EAGLE design)
At the start: 40.8 x 31.7 mm, 13 parts, among them IC2 DS2482-100S, IC3 DS18B20

Commit message: updates
Parts:
- removed A2: (no value), SparkFun-Retired:SJ_3
- removed IC3: DS18B20, 1wire:TO92-
- added IC1: DS18S20, 1wire:TO92-
- moved C1 2.54 mm to (3.05, 12.7), turned to 270 degrees
Connections:
- removed net N$1: A2.2, C1.2
- net 1W: now also IC1.2; no longer IC3.2
- net 5V: no longer A2.1
- net GND: now also IC1.1; no longer IC3.1
- net VDD: now also C1.2, IC1.3; no longer A2.3, IC3.3
Routing:
- net 5V: track 0.00 -> 36.2 mm, vias 0 -> 1
- net 1W: track 0.00 -> 30.0 mm
- net N$5: track 0.00 -> 21.3 mm
- net N$2: track 0.00 -> 20.5 mm, vias 0 -> 1
- net VDD: track 0.00 -> 19.2 mm, vias 0 -> 1
- net N$19: track 0.00 -> 16.3 mm
- net N$21: track 0.00 -> 15.9 mm
- net N$4: track 0.00 -> 11.4 mm
- net N$20: track 0.00 -> 9.91 mm, vias 0 -> 1
- net N$7: track 0.00 -> 7.95 mm
- net N$6: track 0.00 -> 7.23 mm
Other:
- board text added: "Rev C"
- board text removed: "Rev B"
