File: DS2482 1 Wire Controller/Ds2482/DS2482 1 Wire Controller Rev C.sch (EAGLE design)
At the start: 13 parts, among them IC2 DS2482-100S, IC3 DS18B20

Commit message: updates
Parts:
- removed A2: (no value), SparkFun-Retired:SOLDERJUMPER_2WAYS
- removed IC3: DS18B20, 1wire:DS18B20
- added IC1: DS18S20, 1wire:DS18S20
Connections:
- removed net N$1: A2.2, C1.2
- net 5V: no longer A2.1
- net VDD: now also C1.2; no longer A2.3
Changed lines of the file:
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@@
 <grid distance="0.1" unitdist="inch" unit="inch" style="lines" multiple="1" display="no" altdistance="0.01" altunitdist="inch" altunit="inch"/>
 <layers>
-<layer number="1" name="Top" color="4" fill="1" visible="yes" active="no"/>
-<layer number="16" name="Bottom" color="1" fill="1" visible="yes" active="no"/>
-<layer number="17" name="Pads" color="2" fill="1" visible="yes" active="no"/>
-<layer number="18" name="Vias" color="2" fill="1" visible="yes" active="no"/>
-<layer number="19" name="Unrouted" color="6" fill="1" visible="yes" active="no"/>
-<layer number="20" name="Dimension" color="15" fill="1" visible="yes" active="no"/>
-<layer number="21" name="tPlace" color="7" fill="1" visible="yes" active="no"/>
-<layer number="22" name="bPlace" color="7" fill="1" visible="yes" active="no"/>
-<layer number="23" name="tOrigins" color="15" fill="1" visible="yes" active="no"/>
-<layer number="24" name="bOrigins" color="15" fill="1" visible="yes" active="no"/>
-<layer number="25" name="tNames" color="7" fill="1" visible="yes" active="no"/>
-<layer number="26" name="bNames" color="7" fill="1" visible="yes" active="no"/>
-<layer number="27" name="tValues" color="7" fill="1" visible="yes" active="no"/>
-<layer number="28" name="bValues" color="7" fill="1" visible="yes" active="no"/>
+<layer number="1" name="Top" color="4" fill="1" visible="no" active="no"/>
+<layer number="16" name="Bottom" color="1" fill="1" visible="no" active="no"/>
+<layer number="17" name="Pads" color="2" fill="1" visible="no" active="no"/>
+<layer number="18" name="Vias" color="2" fill="1" visible="no" active="no"/>
+<layer number="19" name="Unrouted" color="6" fill="1" visible="no" active="no"/>
+<layer number="20" name="Dimension" color="15" fill="1" visible="no" active="no"/>
+<layer number="21" name="tPlace" color="7" fill="1" visible="no" active="no"/>
+<layer number="22" name="bPlace" color="7" fill="1" visible="no" active="no"/>
+<layer number="23" name="tOrigins" color="15" fill="1" visible="no" active="no"/>
+<layer number="24" name="bOrigins" color="15" fill="1" visible="no" active="no"/>
+<layer number="25" name="tNames" color="7" fill="1" visible="no" active="no"/>
+<layer number="26" name="bNames" color="7" fill="1" visible="no" active="no"/>
+<layer number="27" name="tValues" color="7" fill="1" visible="no" active="no"/>
+<layer number="28" name="bValues" color="7" fill="1" visible="no" active="no"/>
 <layer number="29" name="tStop" color="7" fill="1" visible="no" active="no"/>
 <layer number="30" name="bStop" color="7" fill="1" visible="no" active="no"/>
@@
 <layer number="35" name="tGlue" color="7" fill="4" visible="no" active="no"/>
 <layer number="36" name="bGlue" color="7" fill="5" visible="no" active="no"/>
-<layer number="37" name="tTest" color="7" fill="1" visible="yes" active="no"/>
-<layer number="38" name="bTest" color="7" fill="1" visible="yes" active="no"/>
+<layer number="37" name="tTest" color="7" fill="1" visible="no" active="no"/>
+<layer number="38" name="bTest" color="7" fill="1" visible="no" active="no"/>
 <layer number="39" name="tKeepout" color="4" fill="11" visible="no" active="no"/>
 <layer number="40" name="bKeepout" color="1" fill="11" visible="no" active="no"/>
@@
 <layer number="44" name="Drills" color="7" fill="1" visible="no" active="no"/>
 <layer number="45" name="Holes" color="7" fill="1" visible="no" active="no"/>
-<layer number="46" name="Milling" color="3" fill="1" visible="yes" active="no"/>
-<layer number="47" name="Measures" color="7" fill="1" visible="yes" active="no"/>
-<layer number="48" name="Document" color="7" fill="1" visible="yes" active="no"/>
-<layer number="49" name="Reference" color="7" fill="1" visible="yes" active="no"/>
-<layer number="50" name="dxf" color="7" fill="1" visible="yes" active="no"/>
-<layer number="51" name="tDocu" color="7" fill="1" visible="yes" active="no"/>
-<layer number="52" name="bDocu" color="7" fill="1" visible="yes" active="no"/>
-<layer number="53" name="tGND_GNDA" color="7" fill="9" visible="yes" active="no"/>
-<layer number="54" name="bGND_GNDA" color="1" fill="9" visible="yes" active="no"/>
-<layer number="56" name="wert" color="7" fill="1" visible="yes" active="no"/>
-<layer number="57" name="tCAD" color="7" fill="1" visible="yes" active="no"/>
+<layer number="46" name="Milling" color="3" fill="1" visible="no" active="no"/>
+<layer number="47" name="Measures" color="7" fill="1" visible="no" active="no"/>
+<layer number="48" name="Document" color="7" fill="1" visible="no" active="no"/>
+<layer number="49" name="Reference" color="7" fill="1" visible="no" active="no"/>
+<layer number="50" name="dxf" color="7" fill="1" visible="no" active="no"/>
+<layer number="51" name="tDocu" color="7" fill="1" visible="no" active="no"/>
+<layer number="52" name="bDocu" color="7" fill="1" visible="no" active="no"/>
+<layer number="53" name="tGND_GNDA" color="7" fill="9" visible="no" active="no"/>
+<layer number="54" name="bGND_GNDA" color="1" fill="9" visible="no" active="no"/>
+<layer number="56" name="wert" color="7" fill="1" visible="no" active="no"/>
+<layer number="57" name="tCAD" color="7" fill="1" visible="no" active="no"/>
 <layer number="90" name="Modules" color="5" fill="1" visible="yes" active="yes"/>
 <layer number="91" name="Nets" color="2" fill="1" visible="yes" active="yes"/>
@@
 <part name="SUPPLY2" library="SparkFun-Aesthetics" deviceset="5V" device=""/>
 <part name="IC2" library="1wire" deviceset="DS2482-100" device="S"/>
-<part name="IC3" library="1wire" deviceset="DS18B20" device=""/>
 <part name="JP2" library="SparkFun-Connectors" deviceset="M04" device="PTH"/>
 <part name="GND1" library="SparkFun-Aesthetics" deviceset="GND" device=""/>
@@
 <part name="5VDC1" library="SparkFun-Connectors" deviceset="M02" device="PTH" value="+"/>
 <part name="IO-2" library="SparkFun-Connectors" deviceset="M03" device="PTH"/>
-<part name="A2" library="SparkFun-Retired" deviceset="SOLDERJUMPER_2WAY" device="S"/>
-<part name="SUPPLY3" library="SparkFun-Aesthetics" deviceset="5V" device=""/>
+<part name="IC1" library="1wire" deviceset="DS18S20" device=""/>
 </parts>
 <sheets>
@@
 <instance part="SUPPLY2" gate="G$1" x="78.74" y="170.18"/>
 <instance part="IC2" gate="G$1" x="109.22" y="172.72"/>
-<instance part="IC3" gate="A" x="93.98" y="200.66"/>
 <instance part="JP2" gate="G$1" x="45.72" y="175.26"/>
 <instance part="GND1" gate="1" x="55.88" y="154.94"/>
@@
 <instance part="5VDC1" gate="G$1" x="187.96" y="198.12" rot="R180"/>
 <instance part="IO-2" gate="G$1" x="170.18" y="152.4" rot="R180"/>
-<instance part="A2" gate="G$1" x="58.42" y="200.66" rot="R270"/>
-<instance part="SUPPLY3" gate="G$1" x="68.58" y="200.66"/>
+<instance part="IC1" gate="A" x="99.06" y="205.74"/>
 </instances>
 <busses>
@@
 </net>
 <net name="5V" class="0">
-<segment>
-<pinref part="C1" gate="G$1" pin="1"/>
-<pinref part="SUPPLY1" gate="G$1" pin="5V"/>
-<wire x1="58.42" y1="220.98" x2="58.42" y2="228.6" width="0.1524" layer="91"/>
-</segment>
 <segment>
 <pinref part="SUPPLY2" gate="G$1" pin="5V"/>
@@
 </segment>
 <segment>
-<pinref part="A2" gate="G$1" pin="1"/>
-<wire x1="63.5" y1="200.66" x2="68.58" y2="200.66" width="0.1524" layer="91"/>
-<pinref part="SUPPLY3" gate="G$1" pin="5V"/>
+<pinref part="C1" gate="G$1" pin="1"/>
+<pinref part="SUPPLY1" gate="G$1" pin="5V"/>
+<wire x1="58.42" y1="220.98" x2="58.42" y2="228.6" width="0.1524" layer="91"/>
 </segment>
 </net>
@@
 </segment>
 </net>
+<net name="VDD" class="0">
+<segment>
+<pinref part="C1" gate="G$1" pin="2"/>
+<wire x1="58.42" y1="213.36" x2="58.42" y2="205.74" width="0.1524" layer="91"/>
+</segment>
+</net>
 <net name="1W" class="0">
 <segment>
-<wire x1="93.98" y1="200.66" x2="127" y2="200.66" width="0.1524" layer="91"/>
+<wire x1="127" y1="205.74" x2="127" y2="170.18" width="0.1524" layer="91"/>
+<pinref part="IC2" gate="G$1" pin="1W"/>
+<wire x1="127" y1="170.18" x2="121.92" y2="170.18" width="0.1524" layer="91"/>
 <pinref part="IO-1" gate="G$1" pin="1"/>
-<pinref part="IC2" gate="G$1" pin="1W"/>
 <wire x1="162.56" y1="170.18" x2="127" y2="170.18" width="0.1524" layer="91"/>
+<wire x1="99.06" y1="205.74" x2="127" y2="205.74" width="0.1524" layer="91"/>
 <pinref part="IO-2" gate="G$1" pin="1"/>
-<wire x1="127" y1="170.18" x2="121.92" y2="170.18" width="0.1524" layer="91"/>
-<wire x1="162.56" y1="154.94" x2="121.92" y2="154.94" width="0.1524" layer="91"/>
-<wire x1="121.92" y1="154.94" x2="121.92" y2="170.18" width="0.1524" layer="91"/>
-<wire x1="127" y1="200.66" x2="127" y2="170.18" width="0.1524" layer="91"/>
-</segment>
-</net>
-<net name="N$1" class="0">
-<segment>
-<pinref part="C1" gate="G$1" pin="2"/>
-<pinref part="A2" gate="G$1" pin="2"/>
-<wire x1="58.42" y1="213.36" x2="58.42" y2="205.74" width="0.1524" layer="91"/>
-</segment>
-</net>
-<net name="VDD" class="0">
-<segment>
-<pinref part="A2" gate="G$1" pin="3"/>
-<wire x1="53.34" y1="200.66" x2="45.72" y2="200.66" width="0.1524" layer="91"/>
-</segment>
-</net>
+<wire x1="162.56" y1="154.94" x2="127" y2="154.94" width="0.1524" layer="91"/>
+<wire x1="127" y1="154.94" x2="127" y2="170.18" width="0.1524" layer="91"/>
+</segment>
+</net>
