File: Hive Monitor/Main Board.brd (EAGLE design)
At the start: 113 x 60.6 mm, 80 parts, among them IC1 PCF8574T, IC2 PCF8574T, IC3 PCF8574T, J1 POWER_JACKPTH, Q3 MPS2907A, U1 SI2301BDS-T1-E3, U2 SI2301BDS-T1-E3

Commit message: sync
Parts:
- added 3.3V, CE, CSN, CS_SD, IRQ, MISO, MOSI: TPSB1,27, testpad:B1,27
- added 5V_, SCK, SCL, SDA: SCK, testpad:B1,27
- added GND_: GND, testpad:B1,27
- flipped R10 to the bottom
- flipped R9 to the bottom
Connections:
- new net N$36: CSN.TP, U$3.CSN
- net 3.3V: now also 3.3V.TP
- net 5V: now also 5V_.TP
- net CE_RADIO: now also CE.TP
- net CS-SD: now also CS_SD.TP
- net CSN: no longer U$3.CSN
- net GND: now also GND_.TP
- net IRQ: now also IRQ.TP
- net MISO: now also MISO.TP
- net MOSI: now also MOSI.TP
- net SCK: now also SCK.TP
- net SCL: now also SCL.TP
- net SDA: now also SDA.TP
Routing:
- net CSN: track 64.2 -> 0.00 mm
- net N$36: track 0.00 -> 48.4 mm
- net 3.3V: track 33.2 -> 57.0 mm, vias 0 -> 1
- net 5V: track 311.8 -> 330.0 mm, vias 1 -> 3
- net SCK: track 66.6 -> 80.2 mm
- net CE_RADIO: track 65.9 -> 79.4 mm, vias 0 -> 2
- net ONBOARD: track 107.5 -> 120.0 mm
- net N$31: track 56.9 -> 46.0 mm
- net MOSI: track 67.6 -> 77.8 mm, vias 0 -> 1
- net SCL: track 172.4 -> 182.4 mm
- net N$26: track 29.1 -> 20.4 mm, vias 0 -> 2
- net N$5: track 10.8 -> 19.4 mm
- net IRQ: track 65.0 -> 71.2 mm
- net N$12: track 78.2 -> 72.1 mm, vias 1 -> 2
- net A0: track 80.2 -> 74.1 mm, vias 2 -> 1
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