File: Hive Monitor/Main Board.sch (EAGLE design)
At the start: 80 parts, among them IC1 PCF8574T, IC2 PCF8574T, IC3 PCF8574T, J1 POWER_JACKPTH, Q3 MPS2907A, U1 SI2301BDS-T1-E3, U2 SI2301BDS-T1-E3

Commit message: sync
Parts:
- added 3.3V, CE, CSN, CS_SD, IRQ, MISO, MOSI: TPSB1,27, testpad:TPSB1,27
- added 5V_, SCK, SCL, SDA: SCK, testpad:TPSB1,27
- added GND_: GND, testpad:TPSB1,27
Connections:
- new net N$36: CSN.PP, U$3.CSN
- net 3.3V: now also 3.3V.PP
- net 5V: now also 5V_.PP
- net CE_RADIO: now also CE.PP
- net CS-SD: now also CS_SD.PP
- net CSN: no longer U$3.CSN
- net GND: now also GND_.PP
- net IRQ: now also IRQ.PP
- net MISO: now also MISO.PP
- net MOSI: now also MOSI.PP
- net SCK: now also SCK.PP
- net SCL: now also SCL.PP
- net SDA: now also SDA.PP
