File: Hive Server/Hive Server - Electron.brd (EAGLE design)
At the start: 54.6 x 64.4 mm, 24 parts, among them J1 POWER_JACKPTH

Commit message: sync
Parts:
- removed Q4: (no value), SparkFun-DiscreteSemi:TO-92-AMMO
- removed R16: 100k, SparkFun-Resistors:1/6W-RES
- removed R23: 4.7k, SparkFun-Resistors:1/6W-RES
- removed R32: 300k, SparkFun-Resistors:1/6W-RES
- added C1: 0.1uF, SparkFun-Capacitors:0805
- added CURRENT-MONITOR: (no value), SparkFun-Connectors:1X02
- added R15: 30k, SparkFun-Resistors:1/6W-RES
- added R17: 10k, SparkFun-Resistors:1/6W-RES
- added R7: 300k, SparkFun-Resistors:1/6W-RES
- added U2: SI2301BDS-T1-E3, Vishay_By_element14_Batch_1:SOT95P237X112-3N
- moved R8 33.6 mm to (14.0, 53.3), flipped to the bottom
- moved R9 32.9 mm to (14.0, 49.5), flipped to the bottom
- moved R10 32.4 mm to (14.0, 45.7), flipped to the bottom
- moved R5 26.2 mm to (44.5, 31.8), flipped to the bottom
- moved R2 25.4 mm to (38.1, 35.6), flipped to the bottom
- moved SW2 23.4 mm to (43.2, 11.4)
- moved R6 22.9 mm to (44.5, 35.6), flipped to the bottom
- moved D1 21.6 mm to (-1.27, 14.0), turned to 90 degrees
- moved R1 20.1 mm to (38.1, 31.8), flipped to the bottom
- moved F1 18.1 mm to (3.56, 18.9)
- moved U$8 13.3 mm to (25.1, 9.78)
- moved C4 10.4 mm to (18.9, 45.2), flipped to the bottom, turned to 270 degrees
- moved U$13 10.2 mm to (7.62, 47.0), flipped to the bottom, turned to 90 degrees
- moved C2 3.81 mm to (29.2, 45.7)
- moved R3 3.59 mm to (27.9, 35.6)
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Connections:
- removed net CE_RADIO1: R10.1
- removed net MISO1: R8.1
- removed net MOSI1: R9.1
- removed net N$12: R23.2
- removed net N$17: Q4.2, R23.1
- removed net N$31: Q4.3, R32.1
- removed net S+1: Q4.1
- new net D7: C1.2, U$1.32
- new net N$1: CURRENT-MONITOR.1, D1.C
- new net N$25: C1.1, R7.1, U2.1
- new net N$28: R15.2, U2.3
- net 5V: now also CURRENT-MONITOR.2; no longer D1.C
- net B4: now also R15.1, R17.2; no longer R16.1, R32.2
- net CE_RADIO: now also R10.1
- net GND: now also R17.1; no longer R16.2
- net MISO: now also R8.1
- net MOSI: now also R9.1
- net S+: now also R7.2, U2.2
Routing:
- net 5V: track 0.00 -> 84.7 mm
- net N$4: track 0.00 -> 77.6 mm, vias 0 -> 1
- net SCK: track 0.00 -> 72.9 mm
- net SCL: track 0.00 -> 56.4 mm
- net N$5: track 0.00 -> 56.3 mm, vias 0 -> 2
- net S+: track 0.00 -> 55.6 mm
- net N$6: track 0.00 -> 54.9 mm, vias 0 -> 1
- net SDA: track 0.00 -> 52.0 mm
- net IRQ: track 0.00 -> 51.9 mm, vias 0 -> 1
- net 3.3V: track 0.00 -> 50.5 mm, vias 0 -> 1
- net N$7: track 0.00 -> 49.9 mm, vias 0 -> 1
- net N$1: track 0.00 -> 43.7 mm
- net N$19: track 0.00 -> 37.7 mm
- net MOSI: track 0.00 -> 36.6 mm
- net CSN: track 0.00 -> 26.9 mm
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- added copper zone on layer 1, net GND
- removed copper zone on layer 1, net GND1
Other:
- board size 54.6 x 64.4 mm -> 54.6 x 63.2 mm
- board text added: "ON"
