File: Hive Server/Hive Server - Electron.sch (EAGLE design)
At the start: 24 parts, among them J1 POWER_JACKPTH

Commit message: sync
Parts:
- removed Q4: (no value), SparkFun-DiscreteSemi:TRANSISTOR_NPNBC547
- removed R16: 100k, SparkFun-Resistors:RESISTORPTH-1/6W
- removed R23: 4.7k, SparkFun-Resistors:RESISTORPTH-1/6W
- removed R32: 300k, SparkFun-Resistors:RESISTORPTH-1/6W
- added C1: 0.1uF, SparkFun-Capacitors:2.2UF-25V-+80/-20(0805)
- added CURRENT-MONITOR: M02PTH, SparkFun-Connectors:M02PTH
- added R15: 30k, SparkFun-Resistors:RESISTORPTH-1/6W
- added R17: 10k, SparkFun-Resistors:RESISTORPTH-1/6W
- added R7: 300k, SparkFun-Resistors:RESISTORPTH-1/6W
- added U2: SI2301BDS-T1-E3, Vishay_By_element14_Batch_1:SI2301BDS-T1-E3
Connections:
- removed net CE_RADIO1: R10.1
- removed net MISO1: R8.1
- removed net MOSI1: R9.1
- removed net N$12: R23.2
- removed net N$17: Q4.B, R23.1
- removed net N$31: Q4.E, R32.1
- removed net S+1: Q4.C
- new net D7: C1.2, U$1.D7
- new net N$1: CURRENT-MONITOR.1, D1.C
- new net N$25: C1.1, R7.1, U2.G
- new net N$28: R15.2, U2.D
- net 5V: now also CURRENT-MONITOR.2; no longer D1.C
- net B4: now also R15.1, R17.2; no longer R16.1, R32.2
- net CE_RADIO: now also R10.1
- net GND: now also R17.1; no longer R16.2
- net MISO: now also R8.1
- net MOSI: now also R9.1
- net S+: now also R7.2, U2.S
Other:
- note added: "B4"
- note removed: "A1"
- moved on the sheet: C2, C4, U$7
